Commit message: Task 2.2

File: urdf/differential_robot.urdf (robot description, URDF)
Before this commit: robot three_wheeled_car, 13 links, 12 joints
Links:
- link base_link: mass None -> 0.2; geometry collision cylinder length=0.023999999999999997 radius=0.175; visual cylinder length=0.023999999999999997 radius=0.175
- link head: mass None -> 0.02; geometry collision box size=0.03 0.03 0.03; visual box size=0.03 0.03 0.03
- link left_wheel: mass None -> 0.025; geometry collision cylinder length=0.008 radius=0.036; visual cylinder length=0.008 radius=0.036
- link passive_wheel: mass None -> 0.01; geometry collision sphere radius=0.012; visual sphere radius=0.012
- link passive_wheel_holder: mass None -> 0.015; geometry collision cylinder length=0.011999999999999997 radius=0.012; visual cylinder length=0.011999999999999997 radius=0.012
- link right_wheel: mass None -> 0.025; geometry collision cylinder length=0.008 radius=0.036; visual cylinder length=0.008 radius=0.036
Joints:
- joint base_to_head: origin xyz=0.159 0 0.027 rpy=0 0 0 -> xyz=0.15399999999999997 0 0.026999999999999996 rpy=0 0 0
- joint base_to_passive_wheel_holder: origin xyz=0.162 0 -0.018 rpy=0 0 0 -> xyz=0.15399999999999997 0 -0.017999999999999995 rpy=0 0 0
- joint left_wheel_to_left_wheel_indicator_1: origin xyz=0 -0.031 0.0045 rpy=0 0 0 -> xyz=0 -0.030999999999999996 0.0045000000000000005 rpy=0 0 0
- joint left_wheel_to_left_wheel_indicator_2: origin xyz=0.0268 0.0155 0.0045 rpy=0 0 2.09 -> xyz=0.026846787517317592 0.015500000000000002 0.0045000000000000005 rpy=0 0 2.0943951023931953
- joint left_wheel_to_left_wheel_indicator_3: origin xyz=-0.0268 0.0155 0.0045 rpy=0 0 -2.09 -> xyz=-0.026846787517317592 0.015500000000000002 0.0045000000000000005 rpy=0 0 -2.0943951023931953
- joint passive_wheel_holder_to_passive_wheel: origin xyz=0 0 -0.006 rpy=0 0 0 -> xyz=0 0 -0.005999999999999998 rpy=0 0 0
- joint right_wheel_to_right_wheel_indicator_1: origin xyz=0 -0.031 -0.0045 rpy=0 0 0 -> xyz=0 -0.030999999999999996 -0.0045000000000000005 rpy=0 0 0
- joint right_wheel_to_right_wheel_indicator_2: origin xyz=0.0268 0.0155 -0.0045 rpy=0 0 2.09 -> xyz=0.026846787517317592 0.015500000000000002 -0.0045000000000000005 rpy=0 0 2.0943951023931953
- joint right_wheel_to_right_wheel_indicator_3: origin xyz=-0.0268 0.0155 -0.0045 rpy=0 0 -2.09 -> xyz=-0.026846787517317592 0.015500000000000002 -0.0045000000000000005 rpy=0 0 -2.0943951023931953
